File: slot_8_support_silkscreen.kicad_pcb (KiCad board)
At the start: 2 copper layers, 17.8 x 35.6 mm, 11 parts, among them P6 CONN_1, P7 CONN_1, U1 74LS33

Commit message: Splitting silkscreen/nosilk boards, adding copper pour for mask relief, bottom mask layer
Parts:
- turned C1 to 180 degrees
Routing:
- net VCC: track 27.1 -> 19.6 mm
- added copper zone on F.Cu, net VCC
Other:
- board text removed: "C1"
- board text removed: "R1"
- board text removed: "R2"
- board text removed: "TP1"
- board text removed: "TP2"
- board text removed: "TP3"
- board text removed: "U1"
Changed lines of the file:
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@@
-(kicad_pcb (version 4) (host pcbnew 4.0.0-stable)
+(kicad_pcb (version 4) (host pcbnew 4.0.4-stable)
   (general
     (links 17)
     (no_connects 0)
-    (area 113.882619 89.506428 136.865 128.933571)
+    (area 113.957619 89.581428 136.965 128.858571)
     (thickness 1.6)
-    (drawings 33)
-    (tracks 82)
+    (drawings 24)
+    (tracks 75)
     (zones 0)
     (modules 11)
@@
     (36 B.SilkS user)
     (37 F.SilkS user)
-    (38 B.Mask user)
+    (38 B.Mask user hide)
     (39 F.Mask user)
     (40 Dwgs.User user)
@@
   )
   (setup
-    (last_trace_width 0.3048)
+    (last_trace_width 0.25)
     (user_trace_width 0.1524)
     (user_trace_width 0.2032)
@@
     (visible_elements FFFFFF7F)
     (pcbplotparams
-      (layerselection 0x01080_00000001)
+      (layerselection 0x010e0_00000001)
       (usegerberextensions false)
       (excludeedgelayer true)
@@
       (drillshape 0)
       (scaleselection 1)
-      (outputdirectory gerbers/))
+      (outputdirectory gerbers/silkscreen/))
   )
   (net 0 "")
@@
   )
   (module Capacitors_SMD:C_1206_HandSoldering (layer F.Cu)
-    (at 125.73 95.25)
+    (at 125.73 95.25 180)
     (descr "Capacitor SMD 1206, hand soldering")
     (tags "capacitor 1206")
     (attr smd)
-    (fp_text reference C1 (at -2.54 -1.905) (layer F.SilkS)
-      (effects (font (size 1 1) (thickness 0.15)))
-    )
-    (fp_text value 0.1uF (at 1.27 -1.905) (layer F.SilkS)
+    (fp_text reference C1 (at 2.54 1.905 180) (layer F.SilkS)
+      (effects (font (size 1 1) (thickness 0.15)))
+    )
+    (fp_text value 0.1uF (at -1.27 1.905 180) (layer F.SilkS)
       (effects (font (size 1 1) (thickness 0.15)))
     )
@@
     (fp_line (start 1 -1.025) (end -1 -1.025) (layer F.SilkS) (width 0.15))
     (fp_line (start -1 1.025) (end 1 1.025) (layer F.SilkS) (width 0.15))
-    (pad 1 smd rect (at -2 0) (size 2 1.6) (layers F.Cu F.Paste F.Mask)
+    (pad 1 smd rect (at -2 0 180) (size 2 1.6) (layers F.Cu F.Paste F.Mask)
       (net 1 VCC))
-    (pad 2 smd rect (at 2 0) (size 2 1.6) (layers F.Cu F.Paste F.Mask)
+    (pad 2 smd rect (at 2 0 180) (size 2 1.6) (layers F.Cu F.Paste F.Mask)
       (net 2 GND))
     (model Capacitors_SMD.3dshapes/C_1206_HandSoldering.wrl
@@
       (effects (font (size 1 1) (thickness 0.15)))
     )
-    (fp_text value 74LS33 (at 0 0 450) (layer F.SilkS)
+    (fp_text value 74LS33 (at 0 0 270) (layer F.SilkS) hide
       (effects (font (size 1 1) (thickness 0.15)))
     )
@@
       (net 9 "Net-(/MEMR1-Pad1)"))
   )
+  (gr_text 74LS33 (at 125.73 112.395 270) (layer F.SilkS)
+    (effects (font (size 1.016 1.016) (thickness 0.1778)))
+  )
   (gr_text "Slot 8 Support" (at 120.904 100.33 270) (layer F.SilkS)
     (effects (font (size 1.016 1.016) (thickness 0.1778)))
   )
   (gr_text www.glitchwrks.com/xt-ide (at 130.556 102.362 270) (layer F.SilkS)
-    (effects (font (size 1.016 1.016) (thickness 0.1778)))
-  )
-  (gr_text TP2 (at 120.904 121.412 270) (layer F.Mask)
-    (effects (font (size 1.016 1.016) (thickness 0.1778)))
-  )
-  (gr_text TP3 (at 129.794 124.714 270) (layer F.Mask)
-    (effects (font (size 1.016 1.016) (thickness 0.1778)))
-  )
-  (gr_text TP1 (at 124.968 119.888 270) (layer F.Mask)
-    (effects (font (size 1.016 1.016) (thickness 0.1778)))
-  )
-  (gr_text R1 (at 125.73 97.79) (layer F.Mask)
-    (effects (font (size 1.016 1.016) (thickness 0.1778)))
-  )
-  (gr_text 74LS33 (at 127 111.76 270) (layer F.Mask)
-    (effects (font (size 0.762 0.762) (thickness 0.1778)))
-  )
-  (gr_text U1 (at 125.73 106.68) (layer F.Mask)
-    (effects (font (size 1.016 1.016) (thickness 0.1778)))
-  )
-  (gr_text C1 (at 125.73 93.345) (layer F.Mask)
-    (effects (font (size 1.016 1.016) (thickness 0.1778)))
-  )
-  (gr_text R2 (at 125.73 102.235) (layer F.Mask)
-    (effects (font (size 1.016 1.016) (thickness 0.1778)))
-  )
-  (gr_text "Slot 8 Support" (at 120.904 100.33 270) (layer F.Mask)
-    (effects (font (size 1.016 1.016) (thickness 0.1778)))
-  )
-  (gr_text www.glitchwrks.com/xt-ide (at 130.556 102.362 270) (layer F.Mask)
     (effects (font (size 1.016 1.016) (thickness 0.1778)))
   )
@@
   (gr_line (start 131.826 124.46) (end 131.826 91.44) (angle 90) (layer Edge.Cuts) (width 0.15))
   (gr_line (start 134.62 124.46) (end 131.826 124.46) (angle 90) (layer Edge.Cuts) (width 0.15))
+  (segment (start 127.73 95.25) (end 127.73 92.996) (width 0.8128) (layer F.Cu) (net 1))
+  (segment (start 127.73 92.996) (end 127.762 92.964) (width 0.8128) (layer F.Cu) (net 1))
+  (segment (start 118.11 92.71) (end 120.396 92.71) (width 0.8128) (layer F.Cu) (net 1))
+  (segment (start 127.73 99.695) (end 127.73 95.25) (width 0.8128) (layer F.Cu) (net 1))
   (segment (start 127.73 104.14) (end 127.73 99.695) (width 0.8128) (layer F.Cu) (net 1))
-  (segment (start 127.73 99.695) (end 127.73 97.314) (width 0.8128) (layer F.Cu) (net 1))
-  (segment (start 127.73 97.314) (end 127.698 97.282) (width 0.8128) (layer F.Cu) (net 1))
-  (segment (start 127.698 97.282) (end 125.857 97.282) (width 0.8128) (layer F.Cu) (net 1))
-  (segment (start 123.73 97.25) (end 123.73 95.25) (width 0.8128) (layer F.Cu) (net 1))
-  (segment (start 123.762 97.282) (end 125.857 97.282) (width 0.8128) (layer F.Cu) (net 1))
-  (segment (start 123.73 97.25) (end 123.762 97.282) (width 0.8128) (layer F.Cu) (net 1))
-  (segment (start 123.73 95.25) (end 123.73 92.742) (width 0.8128) (layer F.Cu) (net 1))
-  (segment (start 119.38 92.71) (end 118.11 92.71) (width 0.8128) (layer F.Cu) (net 1))
-  (segment (start 123.698 92.71) (end 119.38 92.71) (width 0.8128) (layer F.Cu) (net 1))
-  (segment (start 123.73 92.742) (end 123.698 92.71) (width 0.8128) (layer F.Cu) (net 1))
   (segment (start 128.778 108.585) (end 127.762 108.585) (width 0.4064) (layer F.Cu) (net 1))
   (segment (start 127.762 108.585) (end 127.73 108.553) (width 0.4064) (layer F.Cu) (net 1))
@@
   (segment (start 127.635 104.775) (end 127.73 104.14) (width 0.4064) (layer F.Cu) (net 1))
   (segment (start 133.35 125.73) (end 130.81 125.73) (width 0.8128) (layer F.Cu) (net 2))
-  (segment (start 130.81 125.73) (end 130.683 125.603) (width 0.8128) (layer F.Cu) (net 2))
   (segment (start 124.206 109.22) (end 121.539 109.22) (width 0.3048) (layer F.Cu) (net 3))
   (segment (start 124.46 109.474) (end 124.206 109.22) (width 0.3048) (layer F.Cu) (net 3))
@@
     (polygon
       (pts
-        (xy 131.826 124.46) (xy 134.493 124.46) (xy 134.493 127) (xy 119.634 126.873) (xy 119.634 91.44)
-        (xy 131.826 91.44) (xy 131.826 124.46)
+        (xy 131.826 124.46) (xy 134.493 124.46) (xy 134.493 127) (xy 119.634 126.873) (xy 119.634 94.488)
+        (xy 122.174 94.488) (xy 122.174 94.742) (xy 129.286 94.742) (xy 129.286 91.44) (xy 131.826 91.44)
       )
     )
+  )
+  (zone (net 1) (net_name VCC) (layer F.Cu) (hatch edge 0.508)
+    (connect_pads (clearance 0.254))
+    (min_thickness 0.254)
+    (fill yes (arc_segments 16) (thermal_gap 0.508) (thermal_bridge_width 0.508))
+    (polygon
+      (pts
+        (xy 128.778 93.98) (xy 119.634 93.98) (xy 119.634 91.44) (xy 128.778 91.44) (xy 128.778 91.694)
+      )
+    )
+  )
+  (zone (net 0) (net_name "") (layer B.Mask) (hatch edge 0.508)
+    (connect_pads (clearance 0.254))
+    (min_thickness 0.254)
+    (fill yes (arc_segments 16) (thermal_gap 0.508) (thermal_bridge_width 0.508))
+    (polygon
+      (pts
+        (xy 131.826 124.46) (xy 134.62 124.46) (xy 134.62 127) (xy 119.634 127) (xy 119.634 114.3)
+        (xy 116.84 114.3) (xy 116.84 111.76) (xy 119.634 111.76) (xy 119.634 109.22) (xy 116.84 109.22)
+        (xy 116.84 106.68) (xy 119.634 106.68) (xy 119.634 93.98) (xy 116.84 93.98) (xy 116.84 91.44)
+        (xy 131.826 91.44)
+      )
+    )
